Commit message: wandb

File: urdf/biped_v4.urdf (robot description, URDF)
Before this commit: robot biped_v4.2, 50 links, 49 joints
Links:
- link base_link: geometry collision mesh filename=/home/control-lab/Desktop/Biped_RL/urdf/meshes/base_link.STL; visual mesh filename=/home/control-lab/Desktop/Biped_RL/urdf/meshes/base_link.STL
- link fix_cfpipe1tobaselink: geometry collision mesh filename=/home/control-lab/Desktop/Biped_RL/urdf/meshes/fix_cfpipe1t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; visual mesh filename=/home/control-lab/Desktop/Biped_RL/urdf/meshes/fix_cfpipe1t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
- link fix_cfpipe2tobaselink: geometry collision mesh filename=/home/control-lab/Desktop/Biped_RL/urdf/meshes/fix_cfpipe2t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; visual mesh filename=/home/control-lab/Desktop/Biped_RL/urdf/meshes/fix_cfpipe2t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
- link fix_femur1_3: geometry collision mesh filename=/home/control-lab/Desktop/Biped_RL/urdf/meshes/fix_femur1_3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; visual mesh filename=/home/control-lab/Desktop/Biped_RL/urdf/meshes/fix_femur1_3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
- link fix_femur1_4: geometry collision mesh filename=/home/control-lab/Desktop/Biped_RL/urdf/meshes/fix_femur1_4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; visual mesh filename=/home/control-lab/Desktop/Biped_RL/urdf/meshes/fix_femur1_4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
- link fix_left_femur2_2: geometry collision mesh filename=/home/control-lab/Desktop/Biped_RL/urdf/meshes/fix_left_fem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; visual mesh filename=/home/control-lab/Desktop/Biped_RL/urdf/meshes/fix_left_fem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
- link fix_left_femur2_3: geometry collision mesh filename=/home/control-lab/Desktop/Biped_RL/urdf/meshes/fix_left_fem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; visual mesh filename=/home/control-lab/Desktop/Biped_RL/urdf/meshes/fix_left_fem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
- link fix_leftfemur1_2: geometry collision mesh filename=/home/control-lab/Desktop/Biped_RL/urdf/meshes/fix_leftfemu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; visual mesh filename=/home/control-lab/Desktop/Biped_RL/urdf/meshes/fix_leftfemu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
- link fix_lefthip1motorbody: geometry collision mesh filename=/home/control-lab/Desktop/Biped_RL/urdf/meshes/fix_lefthip1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; visual mesh filename=/home/control-lab/Desktop/Biped_RL/urdf/meshes/fix_lefthip1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
- link fix_lefthip1towaist: geometry collision mesh filename=/home/control-lab/Desktop/Biped_RL/urdf/meshes/fix_lefthip1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; visual mesh filename=/home/control-lab/Desktop/Biped_RL/urdf/meshes/fix_lefthip1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
- link fix_leftlegtobaselink: geometry collision mesh filename=/home/control-lab/Desktop/Biped_RL/urdf/meshes/fix_leftlegt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; visual mesh filename=/home/control-lab/Desktop/Biped_RL/urdf/meshes/fix_leftlegt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
- link fix_lefttibia_1: geometry collision mesh filename=/home/control-lab/Desktop/Biped_RL/urdf/meshes/fix_lefttibi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; visual mesh filename=/home/control-lab/Desktop/Biped_RL/urdf/meshes/fix_lefttibi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
- link fix_lefttibia_2: geometry collision mesh filename=/home/control-lab/Desktop/Biped_RL/urdf/meshes/fix_lefttibi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; visual mesh filename=/home/control-lab/Desktop/Biped_RL/urdf/meshes/fix_lefttibi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
- link fix_lefttibia_3: geometry collision mesh filename=/home/control-lab/Desktop/Biped_RL/urdf/meshes/fix_lefttibi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; visual mesh filename=/home/control-lab/Desktop/Biped_RL/urdf/meshes/fix_lefttibi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
- link fix_lefttibia_4: geometry collision mesh filename=/home/control-lab/Desktop/Biped_RL/urdf/meshes/fix_lefttibi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; visual mesh filename=/home/control-lab/Desktop/Biped_RL/urdf/meshes/fix_lefttibi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
- link fix_lefttibia_5: geometry collision mesh filename=/home/control-lab/Desktop/Biped_RL/urdf/meshes/fix_lefttibi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; visual mesh filename=/home/control-lab/Desktop/Biped_RL/urdf/meshes/fix_lefttibi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
- link fix_lefttibia_6: geometry collision mesh filename=/home/control-lab/Desktop/Biped_RL/urdf/meshes/fix_lefttibi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; visual mesh filename=/home/control-lab/Desktop/Biped_RL/urdf/meshes/fix_lefttibi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
- link fix_right_femer1_2: geometry collision mesh filename=/home/control-lab/Desktop/Biped_RL/urdf/meshes/fix_right_fe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; visual mesh filename=/home/control-lab/Desktop/Biped_RL/urdf/meshes/fix_right_fe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
- link fix_right_femur2_2: geometry collision mesh filename=/home/control-lab/Desktop/Biped_RL/urdf/meshes/fix_right_fe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; visual mesh filename=/home/control-lab/Desktop/Biped_RL/urdf/meshes/fix_right_fe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
- link fix_right_femur2_3: geometry collision mesh filename=/home/control-lab/Desktop/Biped_RL/urdf/meshes/fix_right_fe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; visual mesh filename=/home/control-lab/Desktop/Biped_RL/urdf/meshes/fix_right_fe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
- link fix_right_hip1motorbody: geometry collision mesh filename=/home/control-lab/Desktop/Biped_RL/urdf/meshes/fix_right_hi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; visual mesh filename=/home/control-lab/Desktop/Biped_RL/urdf/meshes/fix_right_hi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
- link fix_rightfemer1_3: geometry collision mesh filename=/home/control-lab/Desktop/Biped_RL/urdf/meshes/fix_rightfem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; visual mesh filename=/home/control-lab/Desktop/Biped_RL/urdf/meshes/fix_rightfem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
- link fix_rightfemer1_4: geometry collision mesh filename=/home/control-lab/Desktop/Biped_RL/urdf/meshes/fix_rightfem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; visual mesh filename=/home/control-lab/Desktop/Biped_RL/urdf/meshes/fix_rightfem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
- link fix_righthip1towaist: geometry collision mesh filename=/home/control-lab/Desktop/Biped_RL/urdf/meshes/fix_righthip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; visual mesh filename=/home/control-lab/Desktop/Biped_RL/urdf/meshes/fix_righthip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
- link fix_rightlegtobaselink: geometry collision mesh filename=/home/control-lab/Desktop/Biped_RL/urdf/meshes/fix_rightleg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; visual mesh filename=/home/control-lab/Desktop/Biped_RL/urdf/meshes/fix_rightleg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
- link fix_righttibia_1: geometry collision mesh filename=/home/control-lab/Desktop/Biped_RL/urdf/meshes/fix_righttib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; visual mesh filename=/home/control-lab/Desktop/Biped_RL/urdf/meshes/fix_righttib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
- link fix_righttibia_2: geometry collision mesh filename=/home/control-lab/Desktop/Biped_RL/urdf/meshes/fix_righttib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; visual mesh filename=/home/control-lab/Desktop/Biped_RL/urdf/meshes/fix_righttib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
- link fix_righttibia_3: geometry collision mesh filename=/home/control-lab/Desktop/Biped_RL/urdf/meshes/fix_righttib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; visual mesh filename=/home/control-lab/Desktop/Biped_RL/urdf/meshes/fix_righttib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
- link fix_righttibia_4: geometry collision mesh filename=/home/control-lab/Desktop/Biped_RL/urdf/meshes/fix_righttib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; visual mesh filename=/home/control-lab/Desktop/Biped_RL/urdf/meshes/fix_righttib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
- link fix_righttibia_5: geometry collision mesh filename=/home/control-lab/Desktop/Biped_RL/urdf/meshes/fix_righttib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; visual mesh filename=/home/control-lab/Desktop/Biped_RL/urdf/meshes/fix_righttib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
- link fix_righttibia_6: geometry collision mesh filename=/home/control-lab/Desktop/Biped_RL/urdf/meshes/fix_righttib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; visual mesh filename=/home/control-lab/Desktop/Biped_RL/urdf/meshes/fix_righttib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
- link fix_torsolink1: geometry collision mesh filename=/home/control-lab/Desktop/Biped_RL/urdf/meshes/fix_torsolin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; visual mesh filename=/home/control-lab/Desktop/Biped_RL/urdf/meshes/fix_torsolin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
- link fix_torsolink2: geometry collision mesh filename=/home/control-lab/Desktop/Biped_RL/urdf/meshes/fix_torsolin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; visual mesh filename=/home/control-lab/Desktop/Biped_RL/urdf/meshes/fix_torsolin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
- link fix_torsolink3: geometry collision mesh filename=/home/control-lab/Desktop/Biped_RL/urdf/meshes/fix_torsolin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; visual mesh filename=/home/control-lab/Desktop/Biped_RL/urdf/meshes/fix_torsolin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
- link fix_torsotobaselink1: geometry collision mesh filename=/home/control-lab/Desktop/Biped_RL/urdf/meshes/fix_torsotob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; visual mesh filename=/home/control-lab/Desktop/Biped_RL/urdf/meshes/fix_torsotob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
- link fix_torsotobaselink2: geometry collision mesh filename=/home/control-lab/Desktop/Biped_RL/urdf/meshes/fix_torsotob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; visual mesh filename=/home/control-lab/Desktop/Biped_RL/urdf/meshes/fix_torsotob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
- link fix_torsoweight: geometry collision mesh filename=/home/control-lab/Desktop/Biped_RL/urdf/meshes/fix_torsowei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; visual mesh filename=/home/control-lab/Desktop/Biped_RL/urdf/meshes/fix_torsowei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
- link fixed_left_sensor_motor: geometry collision mesh filename=/home/control-lab/Desktop/Biped_RL/urdf/meshes/fixed_left_s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; visual mesh filename=/home/control-lab/Desktop/Biped_RL/urdf/meshes/fixed_left_s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
- link fixed_right_sensor_motor: geometry collision mesh filename=/home/control-lab/Desktop/Biped_RL/urdf/meshes/fixed_right_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; visual mesh filename=/home/control-lab/Desktop/Biped_RL/urdf/meshes/fixed_right_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
- link revolute_left_femur1_1: geometry collision mesh filename=/home/control-lab/Desktop/Biped_RL/urdf/meshes/revolute_lef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; visual mesh filename=/home/control-lab/Desktop/Biped_RL/urdf/meshes/revolute_lef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
- link revolute_left_femur2_1: geometry collision mesh filename=/home/control-lab/Desktop/Biped_RL/urdf/meshes/revolute_lef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; visual mesh filename=/home/control-lab/Desktop/Biped_RL/urdf/meshes/revolute_lef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
- link revolute_left_knee: geometry collision mesh filename=/home/control-lab/Desktop/Biped_RL/urdf/meshes/revolute_lef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; visual mesh filename=/home/control-lab/Desktop/Biped_RL/urdf/meshes/revolute_lef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
- link revolute_left_sensorstick: geometry collision mesh filename=/home/control-lab/Desktop/Biped_RL/urdf/meshes/revolute_lef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; visual mesh filename=/home/control-lab/Desktop/Biped_RL/urdf/meshes/revolute_lef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
- link revolute_leftfoot: geometry collision mesh filename=/home/control-lab/Desktop/Biped_RL/urdf/meshes/revolute_lef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; visual mesh filename=/home/control-lab/Desktop/Biped_RL/urdf/meshes/revolute_lef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
- link revolute_right_femur2_1: geometry collision mesh filename=/home/control-lab/Desktop/Biped_RL/urdf/meshes/revolute_rig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; visual mesh filename=/home/control-lab/Desktop/Biped_RL/urdf/meshes/revolute_rig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
- link revolute_right_knee: geometry collision mesh filename=/home/control-lab/Desktop/Biped_RL/urdf/meshes/revolute_rig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; visual mesh filename=/home/control-lab/Desktop/Biped_RL/urdf/meshes/revolute_rig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
- link revolute_right_sensorstick: geometry collision mesh filename=/home/control-lab/Desktop/Biped_RL/urdf/meshes/revolute_rig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; visual mesh filename=/home/control-lab/Desktop/Biped_RL/urdf/meshes/revolute_rig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
- link revolute_rightfemer1_1: geometry collision mesh filename=/home/control-lab/Desktop/Biped_RL/urdf/meshes/revolute_rig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; visual mesh filename=/home/control-lab/Desktop/Biped_RL/urdf/meshes/revolute_rig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
- link revolute_rightfoot: geometry collision mesh filename=/home/control-lab/Desktop/Biped_RL/urdf/meshes/revolute_rig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; visual mesh filename=/home/control-lab/Desktop/Biped_RL/urdf/meshes/revolute_rig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
- link servo1: geometry collision mesh filename=/home/control-lab/Desktop/Biped_RL/urdf/meshes/servo1.STL; visual mesh filename=/home/control-lab/Desktop/Biped_RL/urdf/meshes/servo1.STL

Commit message: LSTM integration

File: urdf/biped_v4.urdf (robot description, URDF)
Before this commit: robot biped_v4.2, 50 links, 49 joints
Links:
- link base_link: geometry collision mesh filename=/home/samaksh/biped_dev/RLstuff/Biped_RL/urdf/meshes/base_l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; visual mesh filename=/home/samaksh/biped_dev/RLstuff/Biped_RL/urdf/meshes/base_l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
- link fix_cfpipe1tobaselink: geometry collision mesh filename=/home/samaksh/biped_dev/RLstuff/Biped_RL/urdf/meshes/fix_cf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; visual mesh filename=/home/samaksh/biped_dev/RLstuff/Biped_RL/urdf/meshes/fix_cf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
- link fix_cfpipe2tobaselink: geometry collision mesh filename=/home/samaksh/biped_dev/RLstuff/Biped_RL/urdf/meshes/fix_cf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; visual mesh filename=/home/samaksh/biped_dev/RLstuff/Biped_RL/urdf/meshes/fix_cf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
- link fix_femur1_3: geometry collision mesh filename=/home/samaksh/biped_dev/RLstuff/Biped_RL/urdf/meshes/fix_fe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; visual mesh filename=/home/samaksh/biped_dev/RLstuff/Biped_RL/urdf/meshes/fix_fe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
- link fix_femur1_4: geometry collision mesh filename=/home/samaksh/biped_dev/RLstuff/Biped_RL/urdf/meshes/fix_fe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; visual mesh filename=/home/samaksh/biped_dev/RLstuff/Biped_RL/urdf/meshes/fix_fe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
- link fix_left_femur2_2: geometry collision mesh filename=/home/samaksh/biped_dev/RLstuff/Biped_RL/urdf/meshes/fix_le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; visual mesh filename=/home/samaksh/biped_dev/RLstuff/Biped_RL/urdf/meshes/fix_le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
- link fix_left_femur2_3: geometry collision mesh filename=/home/samaksh/biped_dev/RLstuff/Biped_RL/urdf/meshes/fix_le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; visual mesh filename=/home/samaksh/biped_dev/RLstuff/Biped_RL/urdf/meshes/fix_le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
- link fix_leftfemur1_2: geometry collision mesh filename=/home/samaksh/biped_dev/RLstuff/Biped_RL/urdf/meshes/fix_le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; visual mesh filename=/home/samaksh/biped_dev/RLstuff/Biped_RL/urdf/meshes/fix_le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
- link fix_lefthip1motorbody: geometry collision mesh filename=/home/samaksh/biped_dev/RLstuff/Biped_RL/urdf/meshes/fix_le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; visual mesh filename=/home/samaksh/biped_dev/RLstuff/Biped_RL/urdf/meshes/fix_le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
- link fix_lefthip1towaist: geometry collision mesh filename=/home/samaksh/biped_dev/RLstuff/Biped_RL/urdf/meshes/fix_le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; visual mesh filename=/home/samaksh/biped_dev/RLstuff/Biped_RL/urdf/meshes/fix_le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
- link fix_leftlegtobaselink: geometry collision mesh filename=/home/samaksh/biped_dev/RLstuff/Biped_RL/urdf/meshes/fix_le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; visual mesh filename=/home/samaksh/biped_dev/RLstuff/Biped_RL/urdf/meshes/fix_le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
- link fix_lefttibia_1: geometry collision mesh filename=/home/samaksh/biped_dev/RLstuff/Biped_RL/urdf/meshes/fix_le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; visual mesh filename=/home/samaksh/biped_dev/RLstuff/Biped_RL/urdf/meshes/fix_le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
- link fix_lefttibia_2: geometry collision mesh filename=/home/samaksh/biped_dev/RLstuff/Biped_RL/urdf/meshes/fix_le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; visual mesh filename=/home/samaksh/biped_dev/RLstuff/Biped_RL/urdf/meshes/fix_le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
- link fix_lefttibia_3: geometry collision mesh filename=/home/samaksh/biped_dev/RLstuff/Biped_RL/urdf/meshes/fix_le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; visual mesh filename=/home/samaksh/biped_dev/RLstuff/Biped_RL/urdf/meshes/fix_le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
- link fix_lefttibia_4: geometry collision mesh filename=/home/samaksh/biped_dev/RLstuff/Biped_RL/urdf/meshes/fix_le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; visual mesh filename=/home/samaksh/biped_dev/RLstuff/Biped_RL/urdf/meshes/fix_le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
- link fix_lefttibia_5: geometry collision mesh filename=/home/samaksh/biped_dev/RLstuff/Biped_RL/urdf/meshes/fix_le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; visual mesh filename=/home/samaksh/biped_dev/RLstuff/Biped_RL/urdf/meshes/fix_le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
- link fix_lefttibia_6: geometry collision mesh filename=/home/samaksh/biped_dev/RLstuff/Biped_RL/urdf/meshes/fix_le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; visual mesh filename=/home/samaksh/biped_dev/RLstuff/Biped_RL/urdf/meshes/fix_le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
- link fix_right_femer1_2: geometry collision mesh filename=/home/samaksh/biped_dev/RLstuff/Biped_RL/urdf/meshes/fix_ri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; visual mesh filename=/home/samaksh/biped_dev/RLstuff/Biped_RL/urdf/meshes/fix_ri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
- link fix_right_femur2_2: geometry collision mesh filename=/home/samaksh/biped_dev/RLstuff/Biped_RL/urdf/meshes/fix_ri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; visual mesh filename=/home/samaksh/biped_dev/RLstuff/Biped_RL/urdf/meshes/fix_ri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
- link fix_right_femur2_3: geometry collision mesh filename=/home/samaksh/biped_dev/RLstuff/Biped_RL/urdf/meshes/fix_ri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; visual mesh filename=/home/samaksh/biped_dev/RLstuff/Biped_RL/urdf/meshes/fix_ri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
- link fix_right_hip1motorbody: geometry collision mesh filename=/home/samaksh/biped_dev/RLstuff/Biped_RL/urdf/meshes/fix_ri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; visual mesh filename=/home/samaksh/biped_dev/RLstuff/Biped_RL/urdf/meshes/fix_ri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
- link fix_rightfemer1_3: geometry collision mesh filename=/home/samaksh/biped_dev/RLstuff/Biped_RL/urdf/meshes/fix_ri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; visual mesh filename=/home/samaksh/biped_dev/RLstuff/Biped_RL/urdf/meshes/fix_ri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
- link fix_rightfemer1_4: geometry collision mesh filename=/home/samaksh/biped_dev/RLstuff/Biped_RL/urdf/meshes/fix_ri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; visual mesh filename=/home/samaksh/biped_dev/RLstuff/Biped_RL/urdf/meshes/fix_ri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
- link fix_righthip1towaist: geometry collision mesh filename=/home/samaksh/biped_dev/RLstuff/Biped_RL/urdf/meshes/fix_ri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; visual mesh filename=/home/samaksh/biped_dev/RLstuff/Biped_RL/urdf/meshes/fix_ri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
- link fix_rightlegtobaselink: geometry collision mesh filename=/home/samaksh/biped_dev/RLstuff/Biped_RL/urdf/meshes/fix_ri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; visual mesh filename=/home/samaksh/biped_dev/RLstuff/Biped_RL/urdf/meshes/fix_ri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
- link fix_righttibia_1: geometry collision mesh filename=/home/samaksh/biped_dev/RLstuff/Biped_RL/urdf/meshes/fix_ri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; visual mesh filename=/home/samaksh/biped_dev/RLstuff/Biped_RL/urdf/meshes/fix_ri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
- link fix_righttibia_2: geometry collision mesh filename=/home/samaksh/biped_dev/RLstuff/Biped_RL/urdf/meshes/fix_ri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; visual mesh filename=/home/samaksh/biped_dev/RLstuff/Biped_RL/urdf/meshes/fix_ri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
- link fix_righttibia_3: geometry collision mesh filename=/home/samaksh/biped_dev/RLstuff/Biped_RL/urdf/meshes/fix_ri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; visual mesh filename=/home/samaksh/biped_dev/RLstuff/Biped_RL/urdf/meshes/fix_ri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
- link fix_righttibia_4: geometry collision mesh filename=/home/samaksh/biped_dev/RLstuff/Biped_RL/urdf/meshes/fix_ri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; visual mesh filename=/home/samaksh/biped_dev/RLstuff/Biped_RL/urdf/meshes/fix_ri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
- link fix_righttibia_5: geometry collision mesh filename=/home/samaksh/biped_dev/RLstuff/Biped_RL/urdf/meshes/fix_ri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; visual mesh filename=/home/samaksh/biped_dev/RLstuff/Biped_RL/urdf/meshes/fix_ri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
- link fix_righttibia_6: geometry collision mesh filename=/home/samaksh/biped_dev/RLstuff/Biped_RL/urdf/meshes/fix_ri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; visual mesh filename=/home/samaksh/biped_dev/RLstuff/Biped_RL/urdf/meshes/fix_ri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
- link fix_torsolink1: geometry collision mesh filename=/home/samaksh/biped_dev/RLstuff/Biped_RL/urdf/meshes/fix_to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; visual mesh filename=/home/samaksh/biped_dev/RLstuff/Biped_RL/urdf/meshes/fix_to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
- link fix_torsolink2: geometry collision mesh filename=/home/samaksh/biped_dev/RLstuff/Biped_RL/urdf/meshes/fix_to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; visual mesh filename=/home/samaksh/biped_dev/RLstuff/Biped_RL/urdf/meshes/fix_to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
- link fix_torsolink3: geometry collision mesh filename=/home/samaksh/biped_dev/RLstuff/Biped_RL/urdf/meshes/fix_to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; visual mesh filename=/home/samaksh/biped_dev/RLstuff/Biped_RL/urdf/meshes/fix_to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
- link fix_torsotobaselink1: geometry collision mesh filename=/home/samaksh/biped_dev/RLstuff/Biped_RL/urdf/meshes/fix_to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; visual mesh filename=/home/samaksh/biped_dev/RLstuff/Biped_RL/urdf/meshes/fix_to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
- link fix_torsotobaselink2: geometry collision mesh filename=/home/samaksh/biped_dev/RLstuff/Biped_RL/urdf/meshes/fix_to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; visual mesh filename=/home/samaksh/biped_dev/RLstuff/Biped_RL/urdf/meshes/fix_to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
- link fix_torsoweight: geometry collision mesh filename=/home/samaksh/biped_dev/RLstuff/Biped_RL/urdf/meshes/fix_to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; visual mesh filename=/home/samaksh/biped_dev/RLstuff/Biped_RL/urdf/meshes/fix_to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
- link fixed_left_sensor_motor: geometry collision mesh filename=/home/samaksh/biped_dev/RLstuff/Biped_RL/urdf/meshes/fixed_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; visual mesh filename=/home/samaksh/biped_dev/RLstuff/Biped_RL/urdf/meshes/fixed_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
- link fixed_right_sensor_motor: geometry collision mesh filename=/home/samaksh/biped_dev/RLstuff/Biped_RL/urdf/meshes/fixed_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; visual mesh filename=/home/samaksh/biped_dev/RLstuff/Biped_RL/urdf/meshes/fixed_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
- link revolute_left_femur1_1: geometry collision mesh filename=/home/samaksh/biped_dev/RLstuff/Biped_RL/urdf/meshes/revolu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; visual mesh filename=/home/samaksh/biped_dev/RLstuff/Biped_RL/urdf/meshes/revolu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
- link revolute_left_femur2_1: geometry collision mesh filename=/home/samaksh/biped_dev/RLstuff/Biped_RL/urdf/meshes/revolu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; visual mesh filename=/home/samaksh/biped_dev/RLstuff/Biped_RL/urdf/meshes/revolu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
- link revolute_left_knee: geometry collision mesh filename=/home/samaksh/biped_dev/RLstuff/Biped_RL/urdf/meshes/revolu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; visual mesh filename=/home/samaksh/biped_dev/RLstuff/Biped_RL/urdf/meshes/revolu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
- link revolute_left_sensorstick: geometry collision mesh filename=/home/samaksh/biped_dev/RLstuff/Biped_RL/urdf/meshes/revolu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; visual mesh filename=/home/samaksh/biped_dev/RLstuff/Biped_RL/urdf/meshes/revolu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
- link revolute_leftfoot: geometry collision mesh filename=/home/samaksh/biped_dev/RLstuff/Biped_RL/urdf/meshes/revolu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; visual mesh filename=/home/samaksh/biped_dev/RLstuff/Biped_RL/urdf/meshes/revolu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
- link revolute_right_femur2_1: geometry collision mesh filename=/home/samaksh/biped_dev/RLstuff/Biped_RL/urdf/meshes/revolu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; visual mesh filename=/home/samaksh/biped_dev/RLstuff/Biped_RL/urdf/meshes/revolu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
- link revolute_right_knee: geometry collision mesh filename=/home/samaksh/biped_dev/RLstuff/Biped_RL/urdf/meshes/revolu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; visual mesh filename=/home/samaksh/biped_dev/RLstuff/Biped_RL/urdf/meshes/revolu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
- link revolute_right_sensorstick: geometry collision mesh filename=/home/samaksh/biped_dev/RLstuff/Biped_RL/urdf/meshes/revolu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; visual mesh filename=/home/samaksh/biped_dev/RLstuff/Biped_RL/urdf/meshes/revolu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
- link revolute_rightfemer1_1: geometry collision mesh filename=/home/samaksh/biped_dev/RLstuff/Biped_RL/urdf/meshes/revolu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; visual mesh filename=/home/samaksh/biped_dev/RLstuff/Biped_RL/urdf/meshes/revolu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
- link revolute_rightfoot: geometry collision mesh filename=/home/samaksh/biped_dev/RLstuff/Biped_RL/urdf/meshes/revolu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; visual mesh filename=/home/samaksh/biped_dev/RLstuff/Biped_RL/urdf/meshes/revolu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
- link servo1: geometry collision mesh filename=/home/samaksh/biped_dev/RLstuff/Biped_RL/urdf/meshes/servo1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; visual mesh filename=/home/samaksh/biped_dev/RLstuff/Biped_RL/urdf/meshes/servo1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

Commit message: upgraded learning structure

File: urdf/biped_v4.urdf (robot description, URDF)
Before this commit: robot biped_v4.2, 50 links, 49 joints
Joints:
- joint cfpipe1tobaselink: type continuous -> fixed
- joint revolute_torso: axis 1 0 0 -> 0 0 1

Commit message: urdf actuation limits updated

File: urdf/biped_v4.urdf (robot description, URDF)
Before this commit: robot biped_v4.2, 50 links, 49 joints
Joints:
- joint left_ankle: limit lower=-1.732 upper=1.732 effort=1.5 velocity=10 -> lower=-1.732 upper=1.732 effort=1.5 velocity=3
- joint left_hip1: limit lower=-1.732 upper=1.732 effort=3.7 velocity=10 -> lower=-1.732 upper=1.732 effort=4 velocity=2
- joint left_hip2: limit lower=-1.732 upper=1.732 effort=3.7 velocity=10 -> lower=-1.732 upper=1.732 effort=4 velocity=2
- joint left_knee: limit lower=-2 upper=2 effort=5 velocity=10 -> lower=-2 upper=2 effort=4 velocity=2
- joint revolute_torso: limit lower=-1.732 upper=1.732 effort=13 velocity=10 -> lower=-1.732 upper=1.732 effort=4 velocity=2
- joint right_ankle: limit lower=-1.732 upper=1.732 effort=1.5 velocity=10 -> lower=-1.732 upper=1.732 effort=1.5 velocity=2
- joint right_hip1: limit lower=-1.732 upper=1.732 effort=3.7 velocity=10 -> lower=-1.732 upper=1.732 effort=4 velocity=2
- joint right_hip2: limit lower=-1.732 upper=1.732 effort=3.7 velocity=10 -> lower=-1.732 upper=1.732 effort=4 velocity=2
- joint right_knee: limit lower=-2 upper=2 effort=5 velocity=10 -> lower=-2 upper=2 effort=4 velocity=2
