Commit message: urdf file changed the path of stl file to relative

File: urdf/biped_v4.urdf (robot description, URDF)
Before this commit: robot biped_v4.2, 50 links, 49 joints
Links:
- link base_link: geometry collision mesh filename=urdf/meshes/base_link.STL; visual mesh filename=urdf/meshes/base_link.STL
- link fix_cfpipe1tobaselink: geometry collision mesh filename=/urdf/meshes/fix_cfpipe1tobaselink.STL; visual mesh filename=/urdf/meshes/fix_cfpipe1tobaselink.STL
- link fix_cfpipe2tobaselink: geometry collision mesh filename=/urdf/meshes/fix_cfpipe2tobaselink.STL; visual mesh filename=/urdf/meshes/fix_cfpipe2tobaselink.STL
- link fix_femur1_3: geometry collision mesh filename=/urdf/meshes/fix_femur1_3.STL; visual mesh filename=/urdf/meshes/fix_femur1_3.STL
- link fix_femur1_4: geometry collision mesh filename=/urdf/meshes/fix_femur1_4.STL; visual mesh filename=/urdf/meshes/fix_femur1_4.STL
- link fix_left_femur2_2: geometry collision mesh filename=/urdf/meshes/fix_left_femur2_2.STL; visual mesh filename=/urdf/meshes/fix_left_femur2_2.STL
- link fix_left_femur2_3: geometry collision mesh filename=/urdf/meshes/fix_left_femur2_3.STL; visual mesh filename=/urdf/meshes/fix_left_femur2_3.STL
- link fix_leftfemur1_2: geometry collision mesh filename=/urdf/meshes/fix_leftfemur1_2.STL; visual mesh filename=/urdf/meshes/fix_leftfemur1_2.STL
- link fix_lefthip1motorbody: geometry collision mesh filename=/urdf/meshes/fix_lefthip1motorbody.STL; visual mesh filename=/urdf/meshes/fix_lefthip1motorbody.STL
- link fix_lefthip1towaist: geometry collision mesh filename=/urdf/meshes/fix_lefthip1towaist.STL; visual mesh filename=/urdf/meshes/fix_lefthip1towaist.STL
- link fix_leftlegtobaselink: geometry collision mesh filename=/urdf/meshes/fix_leftlegtobaselink.STL; visual mesh filename=/urdf/meshes/fix_leftlegtobaselink.STL
- link fix_lefttibia_1: geometry collision mesh filename=/urdf/meshes/fix_lefttibia_1.STL; visual mesh filename=/urdf/meshes/fix_lefttibia_1.STL
- link fix_lefttibia_2: geometry collision mesh filename=/urdf/meshes/fix_lefttibia_2.STL; visual mesh filename=/urdf/meshes/fix_lefttibia_2.STL
- link fix_lefttibia_3: geometry collision mesh filename=/urdf/meshes/fix_lefttibia_3.STL; visual mesh filename=/urdf/meshes/fix_lefttibia_3.STL
- link fix_lefttibia_4: geometry collision mesh filename=/urdf/meshes/fix_lefttibia_4.STL; visual mesh filename=/urdf/meshes/fix_lefttibia_4.STL
- link fix_lefttibia_5: geometry collision mesh filename=/urdf/meshes/fix_lefttibia_5.STL; visual mesh filename=/urdf/meshes/fix_lefttibia_5.STL
- link fix_lefttibia_6: geometry collision mesh filename=/urdf/meshes/fix_lefttibia_6.STL; visual mesh filename=/urdf/meshes/fix_lefttibia_6.STL
- link fix_right_femer1_2: geometry collision mesh filename=/urdf/meshes/fix_right_femer1_2.STL; visual mesh filename=/urdf/meshes/fix_right_femer1_2.STL
- link fix_right_femur2_2: geometry collision mesh filename=/urdf/meshes/fix_right_femur2_2.STL; visual mesh filename=/urdf/meshes/fix_right_femur2_2.STL
- link fix_right_femur2_3: geometry collision mesh filename=/urdf/meshes/fix_right_femur2_3.STL; visual mesh filename=/urdf/meshes/fix_right_femur2_3.STL
- link fix_right_hip1motorbody: geometry collision mesh filename=/urdf/meshes/fix_right_hip1motorbody.STL; visual mesh filename=/urdf/meshes/fix_right_hip1motorbody.STL
- link fix_rightfemer1_3: geometry collision mesh filename=/urdf/meshes/fix_rightfemer1_3.STL; visual mesh filename=/urdf/meshes/fix_rightfemer1_3.STL
- link fix_rightfemer1_4: geometry collision mesh filename=/urdf/meshes/fix_rightfemer1_4.STL; visual mesh filename=/urdf/meshes/fix_rightfemer1_4.STL
- link fix_righthip1towaist: geometry collision mesh filename=/urdf/meshes/fix_righthip1towaist.STL; visual mesh filename=/urdf/meshes/fix_righthip1towaist.STL
- link fix_rightlegtobaselink: geometry collision mesh filename=/urdf/meshes/fix_rightlegtobaselink.STL; visual mesh filename=/urdf/meshes/fix_rightlegtobaselink.STL
- link fix_righttibia_1: geometry collision mesh filename=/urdf/meshes/fix_righttibia_1.STL; visual mesh filename=/urdf/meshes/fix_righttibia_1.STL
- link fix_righttibia_2: geometry collision mesh filename=/urdf/meshes/fix_righttibia_2.STL; visual mesh filename=/urdf/meshes/fix_righttibia_2.STL
- link fix_righttibia_3: geometry collision mesh filename=/urdf/meshes/fix_righttibia_3.STL; visual mesh filename=/urdf/meshes/fix_righttibia_3.STL
- link fix_righttibia_4: geometry collision mesh filename=/urdf/meshes/fix_righttibia_4.STL; visual mesh filename=/urdf/meshes/fix_righttibia_4.STL
- link fix_righttibia_5: geometry collision mesh filename=/urdf/meshes/fix_righttibia_5.STL; visual mesh filename=/urdf/meshes/fix_righttibia_5.STL
- link fix_righttibia_6: geometry collision mesh filename=/urdf/meshes/fix_righttibia_6.STL; visual mesh filename=/urdf/meshes/fix_righttibia_6.STL
- link fix_torsolink1: geometry collision mesh filename=/urdf/meshes/fix_torsolink1.STL; visual mesh filename=/urdf/meshes/fix_torsolink1.STL
- link fix_torsolink2: geometry collision mesh filename=/urdf/meshes/fix_torsolink2.STL; visual mesh filename=/urdf/meshes/fix_torsolink2.STL
- link fix_torsolink3: geometry collision mesh filename=/urdf/meshes/fix_torsolink3.STL; visual mesh filename=/urdf/meshes/fix_torsolink3.STL
- link fix_torsotobaselink1: geometry collision mesh filename=/urdf/meshes/fix_torsotobaselink1.STL; visual mesh filename=/urdf/meshes/fix_torsotobaselink1.STL
- link fix_torsotobaselink2: geometry collision mesh filename=/urdf/meshes/fix_torsotobaselink2.STL; visual mesh filename=/urdf/meshes/fix_torsotobaselink2.STL
- link fix_torsoweight: geometry collision mesh filename=/urdf/meshes/fix_torsoweight.STL; visual mesh filename=/urdf/meshes/fix_torsoweight.STL
- link fixed_left_sensor_motor: geometry collision mesh filename=/urdf/meshes/fixed_left_sensor_motor.STL; visual mesh filename=/urdf/meshes/fixed_left_sensor_motor.STL
- link fixed_right_sensor_motor: geometry collision mesh filename=/urdf/meshes/fixed_right_sensor_motor.STL; visual mesh filename=/urdf/meshes/fixed_right_sensor_motor.STL
- link revolute_left_femur1_1: geometry collision mesh filename=/urdf/meshes/revolute_left_femur1_1.STL; visual mesh filename=/urdf/meshes/revolute_left_femur1_1.STL
- link revolute_left_femur2_1: geometry collision mesh filename=/urdf/meshes/revolute_left_femur2_1.STL; visual mesh filename=/urdf/meshes/revolute_left_femur2_1.STL
- link revolute_left_knee: geometry collision mesh filename=/urdf/meshes/revolute_left_knee.STL; visual mesh filename=/urdf/meshes/revolute_left_knee.STL
- link revolute_left_sensorstick: geometry collision mesh filename=/urdf/meshes/revolute_left_sensorstick.STL; visual mesh filename=/urdf/meshes/revolute_left_sensorstick.STL
- link revolute_leftfoot: geometry collision mesh filename=/urdf/meshes/revolute_leftfoot.STL; visual mesh filename=/urdf/meshes/revolute_leftfoot.STL
- link revolute_right_femur2_1: geometry collision mesh filename=/urdf/meshes/revolute_right_femur2_1.STL; visual mesh filename=/urdf/meshes/revolute_right_femur2_1.STL
- link revolute_right_knee: geometry collision mesh filename=/urdf/meshes/revolute_right_knee.STL; visual mesh filename=/urdf/meshes/revolute_right_knee.STL
- link revolute_right_sensorstick: geometry collision mesh filename=/urdf/meshes/revolute_right_sensorstick.STL; visual mesh filename=/urdf/meshes/revolute_right_sensorstick.STL
- link revolute_rightfemer1_1: geometry collision mesh filename=/urdf/meshes/revolute_rightfemer1_1.STL; visual mesh filename=/urdf/meshes/revolute_rightfemer1_1.STL
- link revolute_rightfoot: geometry collision mesh filename=/urdf/meshes/revolute_rightfoot.STL; visual mesh filename=/urdf/meshes/revolute_rightfoot.STL
- link servo1: geometry collision mesh filename=/urdf/meshes/servo1.STL; visual mesh filename=/urdf/meshes/servo1.STL

Commit message: urdf changes

File: urdf/biped_v4.urdf (robot description, URDF)
Before this commit: robot biped_v4.2, 50 links, 49 joints
Links:
- link base_link: geometry collision mesh filename=meshes/base_link.STL; visual mesh filename=meshes/base_link.STL
- link fix_cfpipe1tobaselink: geometry collision mesh filename=meshes/fix_cfpipe1tobaselink.STL; visual mesh filename=meshes/fix_cfpipe1tobaselink.STL
- link fix_cfpipe2tobaselink: geometry collision mesh filename=meshes/fix_cfpipe2tobaselink.STL; visual mesh filename=meshes/fix_cfpipe2tobaselink.STL
- link fix_femur1_3: geometry collision mesh filename=meshes/fix_femur1_3.STL; visual mesh filename=meshes/fix_femur1_3.STL
- link fix_femur1_4: geometry collision mesh filename=meshes/fix_femur1_4.STL; visual mesh filename=meshes/fix_femur1_4.STL
- link fix_left_femur2_2: geometry collision mesh filename=meshes/fix_left_femur2_2.STL; visual mesh filename=meshes/fix_left_femur2_2.STL
- link fix_left_femur2_3: geometry collision mesh filename=meshes/fix_left_femur2_3.STL; visual mesh filename=meshes/fix_left_femur2_3.STL
- link fix_leftfemur1_2: geometry collision mesh filename=meshes/fix_leftfemur1_2.STL; visual mesh filename=meshes/fix_leftfemur1_2.STL
- link fix_lefthip1motorbody: geometry collision mesh filename=meshes/fix_lefthip1motorbody.STL; visual mesh filename=meshes/fix_lefthip1motorbody.STL
- link fix_lefthip1towaist: geometry collision mesh filename=meshes/fix_lefthip1towaist.STL; visual mesh filename=meshes/fix_lefthip1towaist.STL
- link fix_leftlegtobaselink: geometry collision mesh filename=meshes/fix_leftlegtobaselink.STL; visual mesh filename=meshes/fix_leftlegtobaselink.STL
- link fix_lefttibia_1: geometry collision mesh filename=meshes/fix_lefttibia_1.STL; visual mesh filename=meshes/fix_lefttibia_1.STL
- link fix_lefttibia_2: geometry collision mesh filename=meshes/fix_lefttibia_2.STL; visual mesh filename=meshes/fix_lefttibia_2.STL
- link fix_lefttibia_3: geometry collision mesh filename=meshes/fix_lefttibia_3.STL; visual mesh filename=meshes/fix_lefttibia_3.STL
- link fix_lefttibia_4: geometry collision mesh filename=meshes/fix_lefttibia_4.STL; visual mesh filename=meshes/fix_lefttibia_4.STL
- link fix_lefttibia_5: geometry collision mesh filename=meshes/fix_lefttibia_5.STL; visual mesh filename=meshes/fix_lefttibia_5.STL
- link fix_lefttibia_6: geometry collision mesh filename=meshes/fix_lefttibia_6.STL; visual mesh filename=meshes/fix_lefttibia_6.STL
- link fix_right_femer1_2: geometry collision mesh filename=meshes/fix_right_femer1_2.STL; visual mesh filename=meshes/fix_right_femer1_2.STL
- link fix_right_femur2_2: geometry collision mesh filename=meshes/fix_right_femur2_2.STL; visual mesh filename=meshes/fix_right_femur2_2.STL
- link fix_right_femur2_3: geometry collision mesh filename=meshes/fix_right_femur2_3.STL; visual mesh filename=meshes/fix_right_femur2_3.STL
- link fix_right_hip1motorbody: geometry collision mesh filename=meshes/fix_right_hip1motorbody.STL; visual mesh filename=meshes/fix_right_hip1motorbody.STL
- link fix_rightfemer1_3: geometry collision mesh filename=meshes/fix_rightfemer1_3.STL; visual mesh filename=meshes/fix_rightfemer1_3.STL
- link fix_rightfemer1_4: geometry collision mesh filename=meshes/fix_rightfemer1_4.STL; visual mesh filename=meshes/fix_rightfemer1_4.STL
- link fix_righthip1towaist: geometry collision mesh filename=meshes/fix_righthip1towaist.STL; visual mesh filename=meshes/fix_righthip1towaist.STL
- link fix_rightlegtobaselink: geometry collision mesh filename=meshes/fix_rightlegtobaselink.STL; visual mesh filename=meshes/fix_rightlegtobaselink.STL
- link fix_righttibia_1: geometry collision mesh filename=meshes/fix_righttibia_1.STL; visual mesh filename=meshes/fix_righttibia_1.STL
- link fix_righttibia_2: geometry collision mesh filename=meshes/fix_righttibia_2.STL; visual mesh filename=meshes/fix_righttibia_2.STL
- link fix_righttibia_3: geometry collision mesh filename=meshes/fix_righttibia_3.STL; visual mesh filename=meshes/fix_righttibia_3.STL
- link fix_righttibia_4: geometry collision mesh filename=meshes/fix_righttibia_4.STL; visual mesh filename=meshes/fix_righttibia_4.STL
- link fix_righttibia_5: geometry collision mesh filename=meshes/fix_righttibia_5.STL; visual mesh filename=meshes/fix_righttibia_5.STL
- link fix_righttibia_6: geometry collision mesh filename=meshes/fix_righttibia_6.STL; visual mesh filename=meshes/fix_righttibia_6.STL
- link fix_torsolink1: geometry collision mesh filename=meshes/fix_torsolink1.STL; visual mesh filename=meshes/fix_torsolink1.STL
- link fix_torsolink2: geometry collision mesh filename=meshes/fix_torsolink2.STL; visual mesh filename=meshes/fix_torsolink2.STL
- link fix_torsolink3: geometry collision mesh filename=meshes/fix_torsolink3.STL; visual mesh filename=meshes/fix_torsolink3.STL
- link fix_torsotobaselink1: geometry collision mesh filename=meshes/fix_torsotobaselink1.STL; visual mesh filename=meshes/fix_torsotobaselink1.STL
- link fix_torsotobaselink2: geometry collision mesh filename=meshes/fix_torsotobaselink2.STL; visual mesh filename=meshes/fix_torsotobaselink2.STL
- link fix_torsoweight: geometry collision mesh filename=meshes/fix_torsoweight.STL; visual mesh filename=meshes/fix_torsoweight.STL
- link fixed_left_sensor_motor: geometry collision mesh filename=meshes/fixed_left_sensor_motor.STL; visual mesh filename=meshes/fixed_left_sensor_motor.STL
- link fixed_right_sensor_motor: geometry collision mesh filename=meshes/fixed_right_sensor_motor.STL; visual mesh filename=meshes/fixed_right_sensor_motor.STL
- link revolute_left_femur1_1: geometry collision mesh filename=meshes/revolute_left_femur1_1.STL; visual mesh filename=meshes/revolute_left_femur1_1.STL
- link revolute_left_femur2_1: geometry collision mesh filename=meshes/revolute_left_femur2_1.STL; visual mesh filename=meshes/revolute_left_femur2_1.STL
- link revolute_left_knee: geometry collision mesh filename=meshes/revolute_left_knee.STL; visual mesh filename=meshes/revolute_left_knee.STL
- link revolute_left_sensorstick: geometry collision mesh filename=meshes/revolute_left_sensorstick.STL; visual mesh filename=meshes/revolute_left_sensorstick.STL
- link revolute_leftfoot: geometry collision mesh filename=meshes/revolute_leftfoot.STL; visual mesh filename=meshes/revolute_leftfoot.STL
- link revolute_right_femur2_1: geometry collision mesh filename=meshes/revolute_right_femur2_1.STL; visual mesh filename=meshes/revolute_right_femur2_1.STL
- link revolute_right_knee: geometry collision mesh filename=meshes/revolute_right_knee.STL; visual mesh filename=meshes/revolute_right_knee.STL
- link revolute_right_sensorstick: geometry collision mesh filename=meshes/revolute_right_sensorstick.STL; visual mesh filename=meshes/revolute_right_sensorstick.STL
- link revolute_rightfemer1_1: geometry collision mesh filename=meshes/revolute_rightfemer1_1.STL; visual mesh filename=meshes/revolute_rightfemer1_1.STL
- link revolute_rightfoot: geometry collision mesh filename=meshes/revolute_rightfoot.STL; visual mesh filename=meshes/revolute_rightfoot.STL
- link servo1: geometry collision mesh filename=meshes/servo1.STL; visual mesh filename=meshes/servo1.STL
